File: PCB/KiCad/TraQAZoid.kicad_sch (KiCad schematic)
At the start: 59 parts, among them SW1 MX_SW_HS, SW10 MX_SW_HS, SW11 MX_SW_HS, SW12 MX_SW_HS, SW13 MX_SW_HS, SW14 MX_SW_HS, SW15 MX_SW_HS, SW16 MX_SW_HS, SW17 MX_SW_HS, SW18 MX_SW_HS, SW19 MX_SW_HS, SW2 MX_SW_HS, SW20 MX_SW_HS, SW21 MX_SW_HS, SW22 MX_SW_HS, SW23 MX_SW_HS, SW24 MX_SW_HS, SW25 MX_SW_HS, SW26 MX_SW_HS, SW27 MX_SW_HS, SW28 MX_SW_HS, SW29 MX_SW_HS, SW3 MX_SW_HS, SW30 MX_SW_HS, SW31 MX_SW_HS, SW32 MX_SW_HS, SW33 MX_SW_HS, SW34 MX_SW_HS, SW35 MX_SW_HS, SW36 MX_SW_HS, SW37 MX_SW_HS, SW4 MX_SW_HS, SW5 MX_SW_HS, SW6 MX_SW_HS, SW7 MX_SW_HS, SW8 MX_SW_HS, SW9 MX_SW_HS, U1 tiny2040

Commit message: Sicherung
Parts:
- S1, S3: footprint marbastlib-mx:STAB_MX_P_6.25u -> marbastlib:STAB_MX_P_2u
- S2: footprint marbastlib-mx:STAB_MX_P_6.25u -> marbastlib:STAB_MX_P_7u
Changed lines of the file:
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@@
       (effects (font (size 1.27 1.27)) (justify left))
     )
-    (property "Footprint" "marbastlib-mx:STAB_MX_P_6.25u" (id 2) (at 137.16 173.99 0)
+    (property "Footprint" "marbastlib:STAB_MX_P_2u" (id 2) (at 137.16 173.99 0)
       (effects (font (size 1.27 1.27)) hide)
     )
@@
       (effects (font (size 1.27 1.27)) (justify left))
     )
-    (property "Footprint" "marbastlib-mx:STAB_MX_P_6.25u" (id 2) (at 93.98 173.99 0)
+    (property "Footprint" "marbastlib:STAB_MX_P_2u" (id 2) (at 93.98 173.99 0)
       (effects (font (size 1.27 1.27)) hide)
     )
@@
       (effects (font (size 1.27 1.27)) (justify left))
     )
-    (property "Footprint" "marbastlib-mx:STAB_MX_P_6.25u" (id 2) (at 116.84 173.99 0)
+    (property "Footprint" "marbastlib:STAB_MX_P_7u" (id 2) (at 116.84 173.99 0)
       (effects (font (size 1.27 1.27)) hide)
     )
@@
     )
     (path "/2d18890b-1c40-40b2-b29a-614110db613d"
-      (reference "S1") (unit 1) (value "MX_stab") (footprint "marbastlib-mx:STAB_MX_P_6.25u")
+      (reference "S1") (unit 1) (value "MX_stab") (footprint "marbastlib:STAB_MX_P_2u")
     )
     (path "/cf92cfbf-bbf9-4882-92bc-563d0035845a"
-      (reference "S2") (unit 1) (value "MX_stab") (footprint "marbastlib-mx:STAB_MX_P_6.25u")
+      (reference "S2") (unit 1) (value "MX_stab") (footprint "marbastlib:STAB_MX_P_7u")
     )
     (path "/16515311-8f86-49e4-bd28-0bf53e99199b"
-      (reference "S3") (unit 1) (value "MX_stab") (footprint "marbastlib-mx:STAB_MX_P_6.25u")
+      (reference "S3") (unit 1) (value "MX_stab") (footprint "marbastlib:STAB_MX_P_2u")
     )
     (path "/bc39e27f-f3e5-40a6-867d-1dd1873b3491"
